Commit message: bilateral teleop script

File: interbotix_ros_xsarms/interbotix_xsarm_descriptions/urdf/wx250s.urdf.xacro (robot description, xacro)
@@ -32,10 +32,10 @@
       <material name="interbotix_black"/>
     </visual>
-    <collision>
+    <!-- <collision>
       <origin rpy="0 0 ${pi/2}" xyz="0 0 0"/>
       <geometry>
         <mesh filename="package://interbotix_xsarm_descriptions/meshes/wx250s_meshes/wx250s_1_base.stl" scale="0.001 0.001 0.001"/>
       </geometry>
-    </collision>
+    </collision> -->
     <inertial>
       <origin rpy="0 0 ${pi/2}" xyz="-0.0380446000 0.0006138920 0.0193354000"/>
@@ -69,10 +69,10 @@
       <material name="interbotix_black"/>
     </visual>
-    <collision>
+    <!-- <collision>
       <origin rpy="0 0 ${pi/2}" xyz="0 0 -0.003"/>
       <geometry>
         <mesh filename="package://interbotix_xsarm_descriptions/meshes/wx250s_meshes/wx250s_2_shoulder.stl" scale="0.001 0.001 0.001"/>
       </geometry>
-    </collision>
+    </collision> -->
     <inertial>
       <origin rpy="0 0 ${pi/2}" xyz="0.0000223482 0.0000414609 0.0066287000"/>
@@ -106,10 +106,10 @@
       <material name="interbotix_black"/>
     </visual>
-    <collision>
+    <!-- <collision>
       <origin rpy="0 0 ${pi/2}" xyz="0 0 0"/>
       <geometry>
         <mesh filename="package://interbotix_xsarm_descriptions/meshes/wx250s_meshes/wx250s_3_upper_arm.stl" scale="0.001 0.001 0.001"/>
       </geometry>
-    </collision>
+    </collision> -->
     <inertial>
       <origin rpy="0 0 ${pi/2}" xyz="0.0171605000 0.0000002725 0.1913230000"/>
@@ -143,10 +143,10 @@
       <material name="interbotix_black"/>
     </visual>
-    <collision>
+    <!-- <collision>
       <origin rpy="0 0 0" xyz="0 0 0"/>
       <geometry>
         <mesh filename="package://interbotix_xsarm_descriptions/meshes/wx250s_meshes/wx250s_4_upper_forearm.stl" scale="0.001 0.001 0.001"/>
       </geometry>
-    </collision>
+    </collision> -->
     <inertial>
       <origin rpy="0 0 0" xyz="0.1079630000 0.0001158760 0"/>
@@ -180,10 +180,10 @@
       <material name="interbotix_black"/>
     </visual>
-    <collision>
+    <!-- <collision>
       <origin rpy="${pi} 0 0" xyz="0 0 0"/>
       <geometry>
         <mesh filename="package://interbotix_xsarm_descriptions/meshes/wx250s_meshes/wx250s_5_lower_forearm.stl" scale="0.001 0.001 0.001"/>
       </geometry>
-    </collision>
+    </collision> -->
     <inertial>
       <origin rpy="${pi} 0 0" xyz="0.0374395000 0.0052225200 0"/>
@@ -217,10 +217,10 @@
       <material name="interbotix_black"/>
     </visual>
-    <collision>
+    <!-- <collision>
       <origin rpy="0 0 ${pi/2}" xyz="0 0 0"/>
       <geometry>
         <mesh filename="package://interbotix_xsarm_descriptions/meshes/wx250s_meshes/wx250s_6_wrist.stl" scale="0.001 0.001 0.001"/>
       </geometry>
-    </collision>
+    </collision> -->
     <inertial>
       <origin rpy="0 0 ${pi/2}" xyz="0.0423600000 -0.0000106630 0.0105770000"/>
@@ -254,10 +254,10 @@
       <material name="interbotix_black"/>
     </visual>
-    <collision>
+    <!-- <collision>
       <origin rpy="0 0 ${pi/2}" xyz="-0.02 0 0"/>
       <geometry>
         <mesh filename="package://interbotix_xsarm_descriptions/meshes/wx250s_meshes/wx250s_7_gripper.stl" scale="0.001 0.001 0.001"/>
       </geometry>
-    </collision>
+    </collision> -->
     <inertial>
       <origin rpy="0 0 ${pi/2}" xyz="0.0216310000 0.0000002516 0.0114100000"/>
@@ -303,10 +303,10 @@
       <material name="interbotix_black"/>
     </visual>
-    <collision>
+    <!-- <collision>
       <origin rpy="0 0 ${pi/2}" xyz="-0.0685 0 0"/>
       <geometry>
         <mesh filename="package://interbotix_xsarm_descriptions/meshes/wx250s_meshes/wx250s_8_gripper_prop.stl" scale="0.001 0.001 0.001"/>
       </geometry>
-    </collision>
+    </collision> -->
     <inertial>
       <origin rpy="0 0 ${pi/2}" xyz="0.0008460000 -0.0000016817 0.0000420000"/>
@@ -331,10 +331,10 @@
         <material name="interbotix_black"/>
       </visual>
-      <collision>
+      <!-- <collision>
         <origin rpy="0 0 0" xyz="0 0 0"/>
         <geometry>
           <mesh filename="package://interbotix_xsarm_descriptions/meshes/wx250s_meshes/wx250s_11_ar_tag.stl" scale="0.001 0.001 0.001"/>
         </geometry>
-      </collision>
+      </collision> -->
       <inertial>
         <origin rpy="0 0 0" xyz="0 0 -0.00315"/>
@@ -360,10 +360,10 @@
         <material name="interbotix_black"/>
       </visual>
-      <collision>
+      <!-- <collision>
         <origin rpy="0 0 ${pi/2}" xyz="-0.063 0 0"/>
         <geometry>
           <mesh filename="package://interbotix_xsarm_descriptions/meshes/wx250s_meshes/wx250s_9_gripper_bar.stl" scale="0.001 0.001 0.001"/>
         </geometry>
-      </collision>
+      </collision> -->
       <inertial>
         <origin rpy="0 0 ${pi/2}" xyz="0.0096870000 0.0000008177 0.0049620000"/>
@@ -411,10 +411,10 @@
           <material name="interbotix_black"/>
         </visual>
-        <collision>
+        <!-- <collision>
           <origin rpy="${pi} ${pi} 0" xyz="0 0.005 0"/>
           <geometry>
             <mesh filename="package://interbotix_xsarm_descriptions/meshes/wx250s_meshes/wx250s_10_gripper_finger.stl" scale="0.001 0.001 0.001"/>
           </geometry>
-        </collision>
+        </collision> -->
         <inertial>
           <origin rpy="${pi} ${pi} ${pi/2}" xyz="0.0138160000 0.0000000000 0.0000000000"/>
@@ -451,10 +451,10 @@
           <material name="interbotix_black"/>
         </visual>
-        <collision>
+        <!-- <collision>
           <origin rpy="0 ${pi} 0" xyz="0 -0.005 0"/>
           <geometry>
             <mesh filename="package://interbotix_xsarm_descriptions/meshes/wx250s_meshes/wx250s_10_gripper_finger.stl" scale="0.001 0.001 0.001"/>
           </geometry>
-        </collision>
+        </collision> -->
         <inertial>
           <origin rpy="0 ${pi} ${pi/2}" xyz="0.0138160000 0.0000000000  0.0000000000"/>
